File: Jadhav/temp.kicad_pcb (KiCad board)
At the start: 2 copper layers, 23 parts, among them SW1 SW_Push, U1 ATmega16A-AU, U2 NCP1117ST33T3G, Y1 8MHz, j1 62910416121

Commit message: Initial PCB layout commit
Routing:
- net GND: track 2.74 -> 167.5 mm, vias 0 -> 1
- net +5: track 1.44 -> 156.9 mm
- net Net-(U1-XTAL1): track 0.00 -> 97.2 mm, vias 0 -> 2
- net /RESET: track 0.00 -> 44.9 mm
- net /MOSI: track 0.33 -> 42.1 mm, vias 0 -> 1
- net /D7: track 0.00 -> 41.0 mm
- net /SCK: track 0.00 -> 40.4 mm
- net Net-(U2-IN): track 0.00 -> 38.4 mm, vias 0 -> 2
- net /MISO: track 0.56 -> 38.4 mm
- net Net-(U1-AREF): track 0.00 -> 37.3 mm, vias 0 -> 2
- net Net-(U1-XTAL2): track 0.00 -> 29.2 mm, vias 0 -> 1
- net /D6: track 0.00 -> 29.1 mm
- net /D5: track 0.00 -> 28.1 mm
- net Net-(U1-PB4_(~{SS})): track 0.00 -> 23.1 mm
- net /D3: track 0.00 -> 21.6 mm
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