File: Jadhav/Jadhav.kicad_sch (KiCad schematic)
At the start: 23 parts, among them SW1 SW_Push, U1 ATmega16A-AU, U2 NCP1117ST33T3G, Y1 8MHz, j1 62910416121

Commit message: Initial PCB layout commit
Parts:
- C1, C2, C3, C5: footprint J_footprint:CAP_9-J_8-E-X_AVX -> J_footprint:G-188_MUR
Other:
- moved on the sheet: g1

Commit message: Updated footprint for LCD
Parts:
- C1, C2, C3, C5: footprint J_footprint:G-188_MUR -> J_footprints:G-188_MUR
- PA1, PB1, PC1, PD1: footprint J_footprint:CONN8_61300811121_WRE -> J_footprints:CONN8_61300811121_WRE
- R3: footprint J_footprint:RES3_PV36W103C01B00_BRN -> J_footprints:RES3_PV36W103C01B00_BRN
- U2: footprint J_footprint:SOT223-3_ONS -> J_footprints:SOT223-3_ONS
- Y1: footprint J_footprint:ATS08A-E_CTS -> J_footprints:ATS08A-E_CTS
- g1, v1: footprint J_footprint:SAMTEC_TS-104-T-AA -> J_footprints:SAMTEC_TS-104-T-AA
- j1: footprint J_footprint:62910416121 -> J_footprints:62910416121
- lcd1: footprint J_footprint:14_CONN_SBH11-PBPC-D07-ST-BK_SUL -> J_footprints:CON14_1X14_TU_HTS_SAI
- prog1: footprint J_footprint:CONN_SBH11-PBPC-D05-ST-BK_SUL -> J_footprints:CONN_SBH11-PBPC-D05-ST-BK_SUL
Changed lines of the file:
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@@
 			)
 		)
-		(property "Footprint" "J_footprint:14_CONN_SBH11-PBPC-D07-ST-BK_SUL"
+		(property "Footprint" "J_footprints:CON14_1X14_TU_HTS_SAI"
 			(at 236.22 173.99 0)
 			(effects
@@
 			)
 		)
-		(property "Footprint" "J_footprint:SOT223-3_ONS"
+		(property "Footprint" "J_footprints:SOT223-3_ONS"
 			(at 226.06 64.77 0)
 			(effects
@@
 			)
 		)
-		(property "Footprint" "J_footprint:CONN8_61300811121_WRE"
+		(property "Footprint" "J_footprints:CONN8_61300811121_WRE"
 			(at 104.14 153.67 0)
 			(effects
@@
 			)
 		)
-		(property "Footprint" "J_footprint:RES3_PV36W103C01B00_BRN"
+		(property "Footprint" "J_footprints:RES3_PV36W103C01B00_BRN"
 			(at 223.52 199.39 0)
 			(effects
@@
 			)
 		)
-		(property "Footprint" "J_footprint:G-188_MUR"
+		(property "Footprint" "J_footprints:G-188_MUR"
 			(at 106.68 201.93 0)
 			(effects
@@
 			)
 		)
-		(property "Footprint" "J_footprint:CONN8_61300811121_WRE"
+		(property "Footprint" "J_footprints:CONN8_61300811121_WRE"
 			(at 246.38 130.81 0)
 			(effects
@@
 			)
 		)
-		(property "Footprint" "J_footprint:ATS08A-E_CTS"
+		(property "Footprint" "J_footprints:ATS08A-E_CTS"
 			(at 114.3 199.39 0)
 			(effects
@@
 			)
 		)
-		(property "Footprint" "J_footprint:CONN8_61300811121_WRE"
+		(property "Footprint" "J_footprints:CONN8_61300811121_WRE"
 			(at 106.68 97.79 0)
 			(effects
@@
 			)
 		)
-		(property "Footprint" "J_footprint:G-188_MUR"
+		(property "Footprint" "J_footprints:G-188_MUR"
 			(at 210.82 181.61 0)
 			(effects
@@
 			)
 		)
-		(property "Footprint" "J_footprint:62910416121"
+		(property "Footprint" "J_footprints:62910416121"
 			(at 185.42 87.63 0)
 			(effects
@@
 			)
 		)
-		(property "Footprint" "J_footprint:G-188_MUR"
+		(property "Footprint" "J_footprints:G-188_MUR"
 			(at 251.46 77.47 0)
 			(effects
@@
 			)
 		)
-		(property "Footprint" "J_footprint:CONN8_61300811121_WRE"
+		(property "Footprint" "J_footprints:CONN8_61300811121_WRE"
 			(at 302.26 107.95 0)
 			(effects
@@
 			)
 		)
-		(property "Footprint" "J_footprint:G-188_MUR"
+		(property "Footprint" "J_footprints:G-188_MUR"
 			(at 116.84 201.93 0)
 			(effects
@@
 			)
 		)
-		(property "Footprint" "J_footprint:CONN_SBH11-PBPC-D05-ST-BK_SUL"
+		(property "Footprint" "J_footprints:CONN_SBH11-PBPC-D05-ST-BK_SUL"
 			(at 72.39 154.94 0)
 			(effects
@@
 			)
 		)
-		(property "Footprint" "J_footprint:SAMTEC_TS-104-T-AA"
+		(property "Footprint" "J_footprints:SAMTEC_TS-104-T-AA"
 			(at 284.48 74.93 0)
 			(effects
@@
 			)
 		)
-		(property "Footprint" "J_footprint:SAMTEC_TS-104-T-AA"
+		(property "Footprint" "J_footprints:SAMTEC_TS-104-T-AA"
 			(at 287.02 90.17 0)
 			(effects

Commit message: Initial routing
Changed lines of the file:
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@@
 	)
 	(junction
+		(at 223.52 161.29)
+		(diameter 0)
+		(color 0 0 0 0)
+	)
+	(junction
 		(at 279.4 69.85)
 		(diameter 0)
@@
 	)
 	(junction
+		(at 154.94 204.47)
+		(diameter 0)
+		(color 0 0 0 0)
+	)
+	(junction
 		(at 294.64 95.25)
 		(diameter 0)
@@
 	(wire
 		(pts
+			(xy 281.94 64.77) (xy 320.04 64.77)
+		)
+		(stroke
+			(width 0)
+			(type default)
+		)
+	)
+	(wire
+		(pts
 			(xy 109.22 140.97) (xy 160.02 140.97)
 		)
@@
 	(wire
 		(pts
-			(xy 289.56 97.79) (xy 312.42 97.79)
+			(xy 313.69 97.79) (xy 313.69 210.82)
+		)
+		(stroke
+			(width 0)
+			(type default)
+		)
+	)
+	(wire
+		(pts
+			(xy 154.94 210.82) (xy 313.69 210.82)
+		)
+		(stroke
+			(width 0)
+			(type default)
+		)
+	)
+	(wire
+		(pts
+			(xy 289.56 97.79) (xy 313.69 97.79)
 		)
 		(stroke
@@
 	(wire
 		(pts
+			(xy 251.46 64.77) (xy 266.7 64.77)
+		)
+		(stroke
+			(width 0)
+			(type default)
+		)
+	)
+	(wire
+		(pts
 			(xy 119.38 181.61) (xy 127 181.61)
 		)
@@
 	(wire
 		(pts
-			(xy 251.46 64.77) (xy 266.7 64.77)
-		)
-		(stroke
-			(width 0)
-			(type default)
-		)
-	)
-	(wire
-		(pts
 			(xy 256.54 196.85) (xy 256.54 179.07)
 		)
@@
 	(wire
 		(pts
+			(xy 320.04 161.29) (xy 223.52 161.29)
+		)
+		(stroke
+			(width 0)
+			(type default)
+		)
+	)
+	(wire
+		(pts
 			(xy 106.68 196.85) (xy 109.22 196.85)
 		)
@@
 	(wire
 		(pts
-			(xy 154.94 196.85) (xy 154.94 176.53)
+			(xy 154.94 176.53) (xy 154.94 196.85)
 		)
 		(stroke
@@
 	(wire
 		(pts
-			(xy 281.94 64.77) (xy 292.1 64.77)
+			(xy 205.74 118.11) (xy 297.18 118.11)
 		)
 		(stroke
@@
 	(wire
 		(pts
-			(xy 205.74 118.11) (xy 297.18 118.11)
+			(xy 127 143.51) (xy 160.02 143.51)
 		)
 		(stroke
@@
 	(wire
 		(pts
-			(xy 127 143.51) (xy 160.02 143.51)
+			(xy 100.33 148.59) (xy 100.33 142.24)
 		)
 		(stroke
@@
 	(wire
 		(pts
-			(xy 100.33 148.59) (xy 100.33 142.24)
+			(xy 236.22 77.47) (xy 246.38 77.47)
 		)
 		(stroke
@@
 	(wire
 		(pts
-			(xy 236.22 77.47) (xy 246.38 77.47)
+			(xy 119.38 181.61) (xy 119.38 191.77)
 		)
 		(stroke
@@
 	(wire
 		(pts
-			(xy 119.38 181.61) (xy 119.38 191.77)
+			(xy 248.92 189.23) (xy 248.92 179.07)
 		)
 		(stroke
@@
 	(wire
 		(pts
-			(xy 248.92 189.23) (xy 248.92 179.07)
+			(xy 154.94 210.82) (xy 154.94 204.47)
 		)
 		(stroke
@@
 	(wire
 		(pts
+			(xy 320.04 64.77) (xy 320.04 161.29)
+		)
+		(stroke
+			(width 0)
+			(type default)
+		)
+	)
+	(wire
+		(pts
 			(xy 238.76 179.07) (xy 238.76 191.77)
 		)
@@
 	(wire
 		(pts
-			(xy 116.84 201.93) (xy 116.84 196.85)
+			(xy 154.94 204.47) (xy 154.94 196.85)
 		)
 		(stroke
@@
 	(wire
 		(pts
-			(xy 154.94 204.47) (xy 154.94 196.85)
+			(xy 116.84 201.93) (xy 116.84 196.85)
 		)
 		(stroke
@@
 	)
 	(symbol
-		(lib_id "Jadhav-altium-import:+5_BAR")
-		(at 292.1 64.77 90)
-		(unit 1)
-		(exclude_from_sim no)
-		(in_bom yes)
-		(on_board yes)
-		(dnp no)
-		(property "Reference" "#PWR0105"
-			(at 292.1 64.77 0)
-			(effects
-				(font
-					(size 1.27 1.27)
-				)
-				(hide yes)
-			)
-		)
-		(property "Value" "+5"
-			(at 295.91 64.77 90)
-			(effects
-				(font
-					(size 1.27 1.27)
-				)
-				(justify right)
-			)
-		)
-		(property "Footprint" ""
-			(at 292.1 64.77 0)
-			(effects
-				(font
-					(size 1.27 1.27)
-				)
-				(hide yes)
-			)
-		)
-		(property "Datasheet" ""
-			(at 292.1 64.77 0)
-			(effects
-				(font
-					(size 1.27 1.27)
-				)
-				(hide yes)
-			)
-		)
-		(property "Description" ""
-			(at 292.1 64.77 0)
-			(effects
-				(font
-					(size 1.27 1.27)
-				)
-				(hide yes)
-			)
-		)
-		(pin ""
-		)
-		(instances
-			(project ""
-				(path "/560f526e-957f-49e1-8860-da49c0378529"
-					(reference "#PWR0105")
-					(unit 1)
-				)
-			)
-		)
-	)
-	(symbol
 		(lib_id "Jadhav-altium-import:GND_POWER_GROUND")
 		(at 111.76 214.63 0)
@@
 					(unit 1)
 				)
-			)
-		)
-	)
-	(symbol
-		(lib_id "Jadhav-altium-import:GND_POWER_GROUND")
-		(at 312.42 97.79 0)
-		(unit 1)
-		(exclude_from_sim no)
-		(in_bom yes)
-		(on_board yes)
-		(dnp no)
-		(property "Reference" "#PWR0104"
-			(at 312.42 97.79 0)
-			(effects
-				(font
-					(size 1.27 1.27)
-				)
-				(hide yes)
-			)
-		)
-		(property "Value" "GND"
-			(at 312.42 104.14 0)
-			(effects
-				(font
-					(size 1.27 1.27)
-				)
-			)
-		)
-		(property "Footprint" ""
-			(at 312.42 97.79 0)
-			(effects
-				(font
-					(size 1.27 1.27)
-				)
-				(hide yes)
-			)
-		)
-		(property "Datasheet" ""
-			(at 312.42 97.79 0)
-			(effects
-				(font
-					(size 1.27 1.27)
-				)
-				(hide yes)
-			)
-		)
-		(property "Description" ""
-			(at 312.42 97.79 0)
-			(effects
-				(font
-					(size 1.27 1.27)
-				)
-				(hide yes)
-			)
-		)
-		(pin ""
-		)
-		(instances
-			(project ""
-				(path "/560f526e-957f-49e1-8860-da49c0378529"
-					(reference "#PWR0104")
-					(unit 1)
-				)

Commit message: g1 v1 fixed
Parts:
- g1, v1: footprint J_footprints:SAMTEC_TS-104-T-AA -> J_footprints:CON4_1X4_TU_HTS_SAI
Changed lines of the file:
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@@
 			)
 		)
-		(property "Footprint" "J_footprints:SAMTEC_TS-104-T-AA"
+		(property "Footprint" "J_footprints:CON4_1X4_TU_HTS_SAI"
 			(at 284.48 74.93 0)
 			(effects
@@
 			)
 		)
-		(property "Footprint" "J_footprints:SAMTEC_TS-104-T-AA"
+		(property "Footprint" "J_footprints:CON4_1X4_TU_HTS_SAI"
 			(at 287.02 90.17 0)
 			(effects
